File: pcb/co2home.kicad_sch (KiCad schematic)
At the start: 9 parts, among them J1 esp32buddy, J2 USB_B_Micro, U1 MH-Z19, U2 TLV75533PDBV, U3 ESP32-WROOM-32D

Commit message: newness
Parts:
- removed C1, C2: 1uF, Capacitor_SMD:C_1206_3216Metric, symbol Device:C_Small
- removed C3: 10uF, Capacitor_SMD:C_1206_3216Metric, symbol Device:C_Small
- removed J1: esp32buddy, Connector_PinHeader_2.54mm:PinHeader_1x06_P2.54mm_Vertical, symbol Connector:Conn_01x06_Socket
- removed J2: USB_B_Micro, !Greg:USB_Micro-B_Amphenol_10103594-0001LF_Horizontal, symbol Connector:USB_B_Micro
- removed R1: 100k, Resistor_SMD:R_1206_3216Metric, symbol Device:R_Small
- removed U1: MH-Z19, !Greg:MH-Z19, symbol !Custom:MH-Z19
- removed U2: TLV75533PDBV, Package_TO_SOT_SMD:SOT-23-5, symbol Regulator_Linear:TLV75533PDBV
- removed U3: ESP32-WROOM-32D, RF_Module:ESP32-WROOM-32D, symbol RF_Module:ESP32-WROOM-32D
- added C1 (x4): 10u, Capacitor_SMD:C_0805_2012Metric, symbol Device:C_Small
- added C5: 0.1u, Capacitor_SMD:C_0603_1608Metric, symbol Device:C_Small
- added H1, H2: MountingHole, MountingHole:MountingHole_3.2mm_M3, symbol Mechanical:MountingHole
- added J2: MH-Z19 L, Connector_PinSocket_2.54mm:PinSocket_1x05_P2.54mm_Vertical, symbol Connector:Conn_01x05_Socket
- added J3: USBC, Connector_USB:USB_C_Receptacle_GCT_USB4105-xx-A_16P_TopMnt_Horizontal, symbol Connector:USB_C_Receptacle_USB2.0
- added J3: eflashy32, Connector_PinHeader_2.54mm:PinHeader_1x06_P2.54mm_Vertical, symbol Connector_Generic:Conn_01x06
- added J4: MH-Z19 R, Connector_PinSocket_2.54mm:PinSocket_1x04_P2.54mm_Vertical, symbol Connector:Conn_01x04_Socket
- added J5: JST-PH, Connector_JST:JST_PH_S7B-PH-SM4-TB_1x07-1MP_P2.00mm_Horizontal, symbol Connector_Generic:Conn_01x07
- added R11, R7 (x2): 10k, Resistor_SMD:R_0402_1005Metric, symbol Device:R_Small
- added R5 (x2): 5k1, Resistor_SMD:R_0402_1005Metric, symbol Device:R_Small
- added SW1: RESET, Button_Switch_SMD:SW_Push_1P1T_XKB_TS-1187A, symbol Switch:SW_SPST
- added U1: ESP32-C3-MINI-1, Espressif:ESP32-C3-MINI-1, symbol Espressif:ESP32-C3-MINI-1
- added U3: AMS1117-3.3, Package_TO_SOT_SMD:SOT-223-3_TabPin2, symbol Regulator_Linear:AP1117-33
Connections:
- net +3V3: now also C1.2, C1.2, C1.2, C5.2, J3.4 (Pin_4), R11.1, R7.1, R7.1, U1.3 (3V3), U3.2 (VO)
- net EN: now also C1.2, J3.5 (Pin_5), R7.2, U1.8 (EN/CHIP_PU)
- net GND: now also C1.1, C1.1, C1.1, C1.1, C5.1, J3.1 (Pin_1), J3.A1 (GND), J3.A12 (GND), J3.B1 (GND), J3.B12 (GND), J4.2 (Pin_2), J5.3 (Pin_3), R5.2, R5.2, SW1.2 (B), U1.1 (GND), U1.11 (GND), U1.14 (GND), U1.2 (GND), U1.36 (GND), U1.37 (GND), U1.38 (GND), U1.39 (GND), U1.40 (GND), U1.41 (GND), U1.42 (GND), U1.43 (GND), U1.44 (GND), U1.45 (GND), U1.46 (GND), U1.47 (GND), U1.48 (GND), U1.49 (GND), U1.50 (GND), U1.51 (GND), U1.52 (GND), U1.53 (GND), U3.1 (GND)
- net GPIO0: now also J3.6 (Pin_6), SW1.1 (A), U1.23 (GPIO9)
- net RXD: now also J2.3 (Pin_3), J5.5 (Pin_5), U1.18 (GPIO4/ADC1_CH4)
- net TXD: now also J2.2 (Pin_2), J5.6 (Pin_6), U1.19 (GPIO5/ADC2_CH0)
- new net: J3.B5 (CC2), R5.1
- new net: J3.A5 (CC1), R5.1
- new net: R11.2, U1.22 (GPIO8)
- new net: R7.2, U1.5 (GPIO2/ADC1_CH2)
- new net +5V: J3.A4 (VBUS), J3.A9 (VBUS), J3.B4 (VBUS), J3.B9 (VBUS), J4.1 (Pin_1), J5.4 (Pin_4), U3.3 (VI)
- new net D+: J3.A6 (D+), J3.B6 (D+), U1.27 (GPIO19/USB_D+)
- new net D-: J3.A7 (D-), J3.B7 (D-), U1.26 (GPIO18/USB_D-)
- new net PROGRXD: J3.3 (Pin_3), U1.30 (GPIO20/U0RXD)
- new net PROGTXD: J3.2 (Pin_2), U1.31 (GPIO21/U0TXD)
- new net PWM: J4.4 (Pin_4), J5.7 (Pin_7), U1.20 (GPIO6)
- no-connect marks 36 -> 14
Other:
- note added: "3V3 Regulation"
- note added: "C3 uses GPIO9 now"
- note added: "ESP32"
- note added: "MH-Z19"
- note added: "Mechanical"
- note added: "Output(TX) from eflashy32"
- note added: "USBC"
- note removed: "(already has small bypass caps)"
- note removed: "34/35 are input only"
- note removed: "Bootstrap GPIO's 0, 2, 5, 12, 15"

Commit message: PN for headers
Parts:
- J2: LCSC (none) -> C50950
- J4: LCSC (none) -> C2718488
Changed lines of the file:
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@@
+      (effects (font (size 1.27 1.27)) hide)
+    )
+    (property "LCSC" "C2718488" (at 105.41 120.65 0)
       (effects (font (size 1.27 1.27)) hide)
     )
@@
       (effects (font (size 1.27 1.27)) hide)
     )
+    (property "LCSC" "C50950" (at 82.55 123.19 0)
+      (effects (font (size 1.27 1.27)) hide)
+    )
